File: Hardware/ARTIC_R2_Module_Breakout.sch (EAGLE design)
At the start: 22 parts, among them U1 2Mbit SPI Flash

Commit message: Final tweaks
Other:
- note added: "2 x PRT-11540"
- note added: "2 x PRT-11541"
- note added: "The ARTIC must be held in reset while programming flash. Use a jumper wire to link RESETB to GND."
- note removed: "The ARTIC must be held in reset while programming flash"
- moved on the sheet: D4, E1, R9, U$22

Commit message: Updates to match the revised module design
Parts:
- removed C2: 22pF, SparkFun-Capacitors:22PF-0402T-16V-10%
- removed C45: 0.1uF, SparkFun-Capacitors:0.1UF-0402T-6.3V-10%-X7R
- removed L1: 30Ω, SparkFun-Coils:FERRITE_BEAD-0402-30OHM-100MHZ
- removed R11, R2: 0, SparkFun-Resistors:0OHM-0402T-1/10W
- removed U$22: ARTIC_R2_MODULE, ARTIC_R2_Module:ARTIC_R2_MODULE
- removed U1: 2Mbit SPI Flash, New_Parts_IC-Memory:SST25VF020BSMD
- added C47: 2.2uF, SparkFun-Capacitors:2.2UF-0402_TIGHT-10V-10%-X5R
- added D5: 1A/23V/620mV, SparkFun-DiscreteSemi:DIODE-SCHOTTKY-BAT20J
- added J2: (no value), Connectors:CONN_06SMD_MALE
- added JP1: JUMPER-SMT_2_NC_TRACE_SILK, SparkFun-Jumpers:JUMPER-SMT_2_NC_TRACE_SILK
- added JP2: JUMPER-SMT_3_1-NC_TRACE_SILK, SparkFun-Jumpers:JUMPER-SMT_3_1-NC_TRACE_SILK
- added Q1: 3.1A/30V/105mΩ, SparkFun-DiscreteSemi:MOSFET_PCH-DMG2307L
- added R10: 100k, SparkFun-Resistors:100KOHM-0402T-1/16W-1%
- added U$3: ARTIC_R2_MODULE, ARTIC_R2_Module:ARTIC_R2_MODULE
- added U8: 3.3V, SparkFun-IC-Power:V_REG_AP2112K-3.3V
- J1: device SparkFun-Connectors:CONN_12SMD_COMBINED -> Connectors:CONN_06SMD_MALE
- J3, J4: device SparkFun-Connectors:CONN_08SMD-COMBO-FEMALE -> Connectors:CONN_08SMD-MALE
Connections:
- removed net FLSH_CEN: U$22.FLSH_CEN, U1.CE
- removed net FLSH_SCLK: U$22.FLSH_SCLK, U1.SCK
- removed net FLSH_SI: U$22.FLSH_SI, U1.SI
- removed net FLSH_SO: U$22.FLSH_SO, U1.SO
- removed net FLSH_VCC: C2.1, C45.1, L1.1, R11.2, R2.2, U1.VCC
- removed net N$1: E1.SIGNAL, U$22.ANTENNA
- removed net N$2: R2.1, U1.HOLD
- removed net N$3: R11.1, U1.WP
- removed net VDD: L1.2, R9.2, U$22.3.3V
- new net 3.3V_OUT: JP1.1, R9.2, U$3.3.3V_OUT
- new net ANTENNA: E1.SIGNAL, U$3.ANTENNA
- new net EN: J2.5, U8.EN
- new net FLASH_PWR: JP1.2, U$3.FLASH_PWR
- new net VCC_1: C47.1, JP2.3, U8.OUT
- new net VCC_2: J4.7, JP2.1
- new net VIN: D5.C, Q1.S, U8.IN
- new net V_BATT: J2.6, Q1.D
- new net V_USB: D5.A, J2.4, Q1.G, R10.2
- net 3.3V: now also JP2.2, U$3.VIN; no longer J4.7, U$22.VIN
- net BOOT: now also U$3.BOOT; no longer U$22.BOOT
- net CIPO: now also U$3.CIPO; no longer U$22.CIPO
- net COPI: now also U$3.COPI; no longer U$22.COPI
- net CS: now also U$3.CS; no longer U$22.CS
- net G8: now also U$3.G8; no longer U$22.G8
- net GND: now also C47.2, R10.1, U$3.GND, U8.GND; no longer C2.2, C45.2, U$22.GND, U1.GND
- net INT1: now also U$3.INT1; no longer U$22.INT1
- net INT2: now also U$3.INT2; no longer U$22.INT2
- net PWR_EN: now also J2.2, U$3.PWR_EN; no longer J1.8, U$22.PWR_EN
- net RESETB: now also J2.1, U$3.RESETB; no longer J1.7, U$22.RESETB
- net SCLK: now also U$3.SCLK; no longer U$22.SCLK
Other:
- note added: "AP2112K-3.3V ------------- Iout (max): 600mA Vin (max): 6.5V Vdrop (max): 250mV Iq: 55uA"
- note added: "Power"
- note removed: "Flash Memory"
- note removed: "The ARTIC must be held in reset while programming flash. Use a jumper wire to link RESETB to GND."
- moved on the sheet: E1, J3, J4
