File: Hardware/Production/ARTIC_R2_Module_Breakout-Panel.brd (EAGLE design)
At the start: 127 x 146.8 mm, 278 parts, among them U1 2Mbit SPI Flash, U2 2Mbit SPI Flash, U3 2Mbit SPI Flash, U4 2Mbit SPI Flash, U5 2Mbit SPI Flash, U6 2Mbit SPI Flash, U7 2Mbit SPI Flash, U8 2Mbit SPI Flash

Commit message: Updates to match the revised module design
Parts:
- removed C10, C12, C14, C8: 22pF, SparkFun-Capacitors:0402-TIGHT
- removed C11, C13, C15, C45, C9: 0.1uF, SparkFun-Capacitors:0402-TIGHT
- removed L1, L2, L3, L4, L5, L6, L7, L8: 30Ω, SparkFun-Coils:0402-TIGHT
- removed R17, R19, R20, R22, R23: 0, SparkFun-Resistors:0402-TIGHT
- removed R18, R21, R24: 1k, SparkFun-Resistors:0402-TIGHT
- added C47: 2.2uF, SparkFun-Capacitors:0402-TIGHT
- added D10, D12, D14, D16: 1A/23V/620mV, SparkFun-DiscreteSemi:SOD-323
- added D11, D13, D15, D9: RED, SparkFun-LED:LED-0603
- added J25, J26, J29, J30: (no value), Connectors:1X08_SMD_MALE
- added J27, J28, J31, J32: (no value), Connectors:1X06_SMD_MALE
- added JP1, JP11, JP13, JP15, JP3, JP5, JP7, JP9: JUMPER-SMT_2_NC_TRACE_SILK, SparkFun-Jumpers:SMT-JUMPER_2_NC_TRACE_SILK
- added JP10, JP12, JP14, JP16, JP2, JP4, JP6, JP8: JUMPER-SMT_3_1-NC_TRACE_SILK, SparkFun-Jumpers:SMT-JUMPER_3_1-NC_TRACE_SILK
- added Q1, Q2, Q3, Q4, Q5, Q6, Q7, Q8: 3.1A/30V/105mΩ, SparkFun-DiscreteSemi:SOT23-3
- added U$121, U$140: (no value), output:#PWR_EN0
- added U$122, U$141: (no value), output:#INT20
- added U$123, U$142: (no value), output:#INT10
- added U$124, U$143: (no value), output:#PWR#0
- added U$125, U$144: (no value), output:ARTIC_R2_BREAKOUT0
- added U$126, U$145: (no value), output:#G8#0
- added U$127, U$146: (no value), output:#GND#0
- added U$128, U$147: (no value), output:#3#3V#0
- added U$129, U$148: ARTIC_R2_MODULE, ARTIC_R2_Module:ARTIC_R2_MODULE
- added U$130, U$149: (no value), output:#VBAT#0
- added U$131, U$150: (no value), output:#EN#0
- added U$132, U$151: (no value), output:#VUSB#0
- added U$133, U$152: (no value), output:#FLASH_PWR#0
- added U$134: (no value), output:CIPO#0
- added U$135: (no value), output:COPI#0
- added U$136: (no value), output:SCLK#0
- added U$137: (no value), output:CS#0
- added U$138: (no value), output:#BOOT0
- added U$139: (no value), output:#RESETB0
- C1, C2, C4, C6: value 22pF -> 2.2uF
- C3, C5, C7: value 0.1uF -> 2.2uF
- D2, D5, D6, D8: value RED -> 1A/23V/620mV; device SparkFun-LED:LED-0603 -> SparkFun-DiscreteSemi:SOD-323
- J1, J16, J19, J2, J7: device SparkFun-Connectors:1X12_SMD_COMBINED -> Connectors:1X06_SMD_MALE
- J10, J13, J22: device SparkFun-Connectors:1X12_SMD_COMBINED -> Connectors:1X08_SMD_MALE
- J11, J12, J15, J20, J23, J24, J8: device SparkFun-Connectors:1X08_SMD_COMBINED -> Connectors:1X06_SMD_MALE
- J14, J17, J18, J21, J3, J4, J5, J6, J9: device SparkFun-Connectors:1X08_SMD_COMBINED -> Connectors:1X08_SMD_MALE
- R1, R11, R13, R3, R5: value 0 -> 1k
- R10, R14, R16, R2, R6, R8: value 0 -> 100k
- R12, R4: value 1k -> 100k
- U$10, U$96: device output:#RESETB0 -> output:CIPO#0
- U$100, U$17: device output:#PWR#0 -> output:#BOOT0
- U$101, U$20: device output:ARTIC_R2_BREAKOUT0 -> output:#RESETB0
- U$102, U$21: device output:#G8#0 -> output:#PWR_EN0
- U$103, U$22: value ARTIC_R2_MODULE -> (none); device ARTIC_R2_Module:ARTIC_R2_MODULE -> output:#INT20
- U$104: device output:#GND#0 -> output:#INT10
- U$105: device output:#3#3V#0 -> output:#PWR#0
- U$106: device output:CIPO#0 -> output:ARTIC_R2_BREAKOUT0
- U$107: device output:COPI#0 -> output:#G8#0
- U$108: device output:SCLK#0 -> output:#GND#0
- U$109: device output:CS#0 -> output:#3#3V#0
- U$11, U$97: device output:#PWR_EN0 -> output:COPI#0
- U$110: value (none) -> ARTIC_R2_MODULE; device output:#BOOT0 -> ARTIC_R2_Module:ARTIC_R2_MODULE
- U$111: device output:#RESETB0 -> output:#VBAT#0
- U$112: device output:#PWR_EN0 -> output:#EN#0
- U$113: device output:#INT20 -> output:#VUSB#0
- U$114: device output:#INT10 -> output:#FLASH_PWR#0
- U$115: device output:#PWR#0 -> output:CIPO#0
- U$116: device output:ARTIC_R2_BREAKOUT0 -> output:COPI#0
- U$117: device output:#G8#0 -> output:SCLK#0
- U$118: value ARTIC_R2_MODULE -> (none); device ARTIC_R2_Module:ARTIC_R2_MODULE -> output:CS#0
- U$119: device output:#GND#0 -> output:#BOOT0
- U$120: device output:#3#3V#0 -> output:#RESETB0
- U$13, U$98: device output:#INT20 -> output:SCLK#0
- U$15, U$99: device output:#INT10 -> output:CS#0
- U$23: value ARTIC_R2_MODULE -> (none); device ARTIC_R2_Module:ARTIC_R2_MODULE -> output:#INT10
- U$27: device output:#GND#0 -> output:#PWR#0
- U$3, U$91: value (none) -> ARTIC_R2_MODULE; device output:CIPO#0 -> ARTIC_R2_Module:ARTIC_R2_MODULE
- U$30: device output:#3#3V#0 -> output:ARTIC_R2_BREAKOUT0
- U$31: device output:CIPO#0 -> output:#G8#0
- U$32: device output:COPI#0 -> output:#GND#0
- U$33: device output:SCLK#0 -> output:#3#3V#0
- U$34: value (none) -> ARTIC_R2_MODULE; device output:CS#0 -> ARTIC_R2_Module:ARTIC_R2_MODULE
- U$35: device output:#BOOT0 -> output:#VBAT#0
- U$36: device output:#RESETB0 -> output:#EN#0
- U$37: device output:#PWR_EN0 -> output:#VUSB#0
- U$38: device output:#INT20 -> output:#FLASH_PWR#0
- U$39: device output:#INT10 -> output:CIPO#0
- U$4: device output:COPI#0 -> output:#FLASH_PWR#0
- U$40: device output:#PWR#0 -> output:COPI#0
- U$41: device output:ARTIC_R2_BREAKOUT0 -> output:SCLK#0
- U$42: device output:#G8#0 -> output:CS#0
- U$43: value ARTIC_R2_MODULE -> (none); device ARTIC_R2_Module:ARTIC_R2_MODULE -> output:#BOOT0
- U$44: device output:#GND#0 -> output:#RESETB0
- U$45: device output:#3#3V#0 -> output:#PWR_EN0
- U$46: device output:CIPO#0 -> output:#INT20
- U$47: device output:COPI#0 -> output:#INT10
- U$48: device output:SCLK#0 -> output:#PWR#0
- U$49: device output:CS#0 -> output:ARTIC_R2_BREAKOUT0
- U$5: device output:SCLK#0 -> output:#VBAT#0
- U$50: device output:#BOOT0 -> output:#G8#0
- U$51: device output:#RESETB0 -> output:#GND#0
- U$52: device output:#PWR_EN0 -> output:#3#3V#0
- U$53: value (none) -> ARTIC_R2_MODULE; device output:#INT20 -> ARTIC_R2_Module:ARTIC_R2_MODULE
- U$54: device output:#INT10 -> output:#VBAT#0
- U$55: device output:#PWR#0 -> output:#EN#0
- U$56: device output:ARTIC_R2_BREAKOUT0 -> output:#VUSB#0
- U$57: device output:#G8#0 -> output:#FLASH_PWR#0
- U$58: value ARTIC_R2_MODULE -> (none); device ARTIC_R2_Module:ARTIC_R2_MODULE -> output:CIPO#0
- U$59: device output:#GND#0 -> output:COPI#0
- U$60: device output:#3#3V#0 -> output:SCLK#0
- U$61: device output:CIPO#0 -> output:CS#0
- U$62: device output:COPI#0 -> output:#BOOT0
- U$63: device output:SCLK#0 -> output:#RESETB0
- U$64: device output:CS#0 -> output:#PWR_EN0
- U$65: device output:#BOOT0 -> output:#INT20
- U$66: device output:#RESETB0 -> output:#INT10
- U$67: device output:#PWR_EN0 -> output:#PWR#0
- U$68: device output:#INT20 -> output:ARTIC_R2_BREAKOUT0
- U$69: device output:#INT10 -> output:#G8#0
- U$7: device output:CS#0 -> output:#EN#0
- U$70: device output:#PWR#0 -> output:#GND#0
- U$71: device output:ARTIC_R2_BREAKOUT0 -> output:#3#3V#0
- U$72: value (none) -> ARTIC_R2_MODULE; device output:#G8#0 -> ARTIC_R2_Module:ARTIC_R2_MODULE
- U$73: value ARTIC_R2_MODULE -> (none); device ARTIC_R2_Module:ARTIC_R2_MODULE -> output:#VBAT#0
- U$74: device output:#GND#0 -> output:#EN#0
- U$75: device output:#3#3V#0 -> output:#VUSB#0
- U$76: device output:CIPO#0 -> output:#FLASH_PWR#0
- U$77: device output:COPI#0 -> output:CIPO#0
- U$78: device output:SCLK#0 -> output:COPI#0
- U$79: device output:CS#0 -> output:SCLK#0
- U$8: device output:#BOOT0 -> output:#VUSB#0
- U$80: device output:#BOOT0 -> output:CS#0
- U$81: device output:#RESETB0 -> output:#BOOT0
- U$82: device output:#PWR_EN0 -> output:#RESETB0
- U$83: device output:#INT20 -> output:#PWR_EN0
- U$84: device output:#INT10 -> output:#INT20
- U$85: device output:#PWR#0 -> output:#INT10
- U$86: device output:ARTIC_R2_BREAKOUT0 -> output:#PWR#0
- U$87: device output:#G8#0 -> output:ARTIC_R2_BREAKOUT0
- U$88: value ARTIC_R2_MODULE -> (none); device ARTIC_R2_Module:ARTIC_R2_MODULE -> output:#G8#0
- U$92: device output:COPI#0 -> output:#VBAT#0
- U$93: device output:SCLK#0 -> output:#EN#0
- U$94: device output:CS#0 -> output:#VUSB#0
- U$95: device output:#BOOT0 -> output:#FLASH_PWR#0
- U1, U2, U3, U4, U5, U6, U7, U8: value 2Mbit SPI Flash -> 3.3V; device New_Parts_IC-Memory:SO08 -> SparkFun-IC-Power:SOT23-5
- moved U$67 122.4 mm to (99.4, 2.54), flipped to the top
- moved J13 121.0 mm to (109.5, 44.5)
- moved U$72 117.6 mm to (99.3, 24.1), flipped to the top
- moved J14 116.5 mm to (109.5, 24.1)
- moved U$71 114.7 mm to (104.3, 8.89), turned to 0 degrees
- moved U$68 114.0 mm to (100.6, 23.5), turned to 90 degrees
- moved U$70 113.4 mm to (104.4, 14.0), flipped to the bottom
- moved R8 109.7 mm to (10.2, 60.2), turned to 180 degrees
- moved U$61 108.7 mm to (105.4, 29.2)
- moved U$65 106.5 mm to (94.0, 31.8)
- moved U$73 104.8 mm to (94.9, 16.5), flipped to the bottom
- moved U4 102.1 mm to (16.6, 63.8)
- moved U8 100.9 mm to (16.6, 4.83)
- moved U$69 100.9 mm to (93.6, 39.4)
- moved U$66 100.1 mm to (93.9, 34.3)
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Connections:
- removed net FLSH_CEN: U$22.20, U1.1
- removed net FLSH_CEN1: U$23.20, U2.1
- removed net FLSH_CEN2: U$43.20, U3.1
- removed net FLSH_CEN3: U$58.20, U4.1
- removed net FLSH_CEN4: U$73.20, U5.1
- removed net FLSH_CEN5: U$88.20, U6.1
- removed net FLSH_CEN6: U$103.20, U7.1
- removed net FLSH_CEN7: U$118.20, U8.1
- removed net FLSH_SCLK: U$22.17, U1.6
- removed net FLSH_SCLK1: U$23.17, U2.6
- removed net FLSH_SCLK2: U$43.17, U3.6
- removed net FLSH_SCLK3: U$58.17, U4.6
- removed net FLSH_SCLK4: U$73.17, U5.6
- removed net FLSH_SCLK5: U$88.17, U6.6
- removed net FLSH_SCLK6: U$103.17, U7.6
- removed net FLSH_SCLK7: U$118.17, U8.6
- removed net FLSH_SI: U$22.18, U1.5
- removed net FLSH_SI1: U$23.18, U2.5
- removed net FLSH_SI2: U$43.18, U3.5
- removed net FLSH_SI3: U$58.18, U4.5
- removed net FLSH_SI4: U$73.18, U5.5
- removed net FLSH_SI5: U$88.18, U6.5
- removed net FLSH_SI6: U$103.18, U7.5
- removed net FLSH_SI7: U$118.18, U8.5
- removed net FLSH_SO: U$22.19, U1.2
- removed net FLSH_SO1: U$23.19, U2.2
- removed net FLSH_SO2: U$43.19, U3.2
- removed net FLSH_SO3: U$58.19, U4.2
- removed net FLSH_SO4: U$73.19, U5.2
- removed net FLSH_SO5: U$88.19, U6.2
- removed net FLSH_SO6: U$103.19, U7.2
- removed net FLSH_SO7: U$118.19, U8.2
- removed net FLSH_VCC: C2.1, C45.1, L1.1, R11.2, R2.2, U1.8
- removed net FLSH_VCC1: C1.1, C3.1, L2.1, R1.2, R3.2, U2.8
- removed net FLSH_VCC2: C4.1, C5.1, L3.1, R5.2, R6.2, U3.8
- removed net FLSH_VCC3: C6.1, C7.1, L4.1, R10.2, R8.2, U4.8
- removed net FLSH_VCC4: C8.1, C9.1, L5.1, R13.2, R14.2, U5.8
- removed net FLSH_VCC5: C10.1, C11.1, L6.1, R16.2, R17.2, U6.8
- removed net FLSH_VCC6: C12.1, C13.1, L7.1, R19.2, R20.2, U7.8
- removed net FLSH_VCC7: C14.1, C15.1, L8.1, R22.2, R23.2, U8.8
- removed net N$10: D2.A, R7.1
- removed net N$11: E3.SIG, U$43.23
- removed net N$12: R8.1, U4.7
- removed net N$13: R10.1, U4.3
- removed net N$14: D3.A, R12.1
- removed net N$15: E4.SIG, U$58.23
- removed net N$16: R13.1, U5.7
- removed net N$17: R14.1, U5.3
- removed net N$18: D5.A, R15.1
- removed net N$19: E5.SIG, U$73.23
- removed net N$20: R16.1, U6.7
- removed net N$21: R17.1, U6.3
- removed net N$23: D6.A, R18.1
- removed net N$24: E6.SIG, U$88.23
- removed net N$25: R19.1, U7.7
- removed net N$26: R20.1, U7.3
- removed net N$27: D7.A, R21.1
- removed net N$28: E7.SIG, U$103.23
- removed net N$29: R22.1, U8.7
- removed net N$30: R23.1, U8.3
- removed net N$31: D8.A, R24.1
- removed net N$32: E8.SIG, U$118.23
- removed net N$8: R5.1, U3.7
- removed net N$9: R6.1, U3.3
- removed net VDD: L1.2, R9.2, U$22.21
- removed net VDD1: L2.2, R4.2, U$23.21
- removed net VDD2: L3.2, R7.2, U$43.21
- removed net VDD3: L4.2, R12.2, U$58.21
- removed net VDD4: L5.2, R15.2, U$73.21
- removed net VDD5: L6.2, R18.2, U$88.21
- removed net VDD6: L7.2, R21.2, U$103.21
- removed net VDD7: L8.2, R24.2, U$118.21
- new net 3.3V_OUT: JP1.1, R9.2, U$3.17
- new net 3.3V_OUT1: JP3.1, R1.2, U$34.17
- new net 3.3V_OUT2: JP5.1, R3.2, U$53.17
- new net 3.3V_OUT3: JP7.1, R5.2, U$72.17
- new net 3.3V_OUT4: JP9.1, R7.2, U$91.17
- new net 3.3V_OUT5: JP11.1, R11.2, U$110.17
- new net 3.3V_OUT6: JP13.1, R13.2, U$129.17
- new net 3.3V_OUT7: JP15.1, R15.2, U$148.17
- new net ANTENNA: E1.SIG, U$3.23
- new net ANTENNA1: E2.SIG, U$34.23
- new net ANTENNA2: E3.SIG, U$53.23
- new net ANTENNA3: E4.SIG, U$72.23
- new net ANTENNA4: E5.SIG, U$91.23
- new net ANTENNA5: E6.SIG, U$110.23
- new net ANTENNA6: E7.SIG, U$129.23
- new net ANTENNA7: E8.SIG, U$148.23
- new net EN: J2.5, U8.3
- new net EN1: J7.5, U1.3
- new net EN2: J11.5, U2.3
- new net EN3: J15.5, U3.3
- new net EN4: J19.5, U4.3
- new net EN5: J23.5, U5.3
- new net EN6: J27.5, U6.3
- new net EN7: J31.5, U7.3
- new net FLASH_PWR: JP1.2, U$3.16
- new net FLASH_PWR1: JP3.2, U$34.16
- new net FLASH_PWR2: JP5.2, U$53.16
- new net FLASH_PWR3: JP7.2, U$72.16
- new net FLASH_PWR4: JP9.2, U$91.16
- new net FLASH_PWR5: JP11.2, U$110.16
- new net FLASH_PWR6: JP13.2, U$129.16
- new net FLASH_PWR7: JP15.2, U$148.16
- new net VCC_1: C47.1, JP2.3, U8.5
- new net VCC_10: J18.7, JP10.1
- new net VCC_11: C5.1, JP12.3, U5.5
- new net VCC_12: J22.7, JP12.1
- new net VCC_13: C6.1, JP14.3, U6.5
- new net VCC_14: J26.7, JP14.1
- new net VCC_15: C7.1, JP16.3, U7.5
- new net VCC_16: J30.7, JP16.1
- new net VCC_2: J4.7, JP2.1
- new net VCC_3: C1.1, JP4.3, U1.5
- new net VCC_4: J6.7, JP4.1
- new net VCC_5: C2.1, JP6.3, U2.5
- new net VCC_6: J10.7, JP6.1
- new net VCC_7: C3.1, JP8.3, U3.5
- new net VCC_8: J14.7, JP8.1
- new net VCC_9: C4.1, JP10.3, U4.5
- new net VIN: D5.C, Q1.2, U8.1
- new net VIN1: D2.C, Q2.2, U1.1
- new net VIN2: D6.C, Q3.2, U2.1
- new net VIN3: D8.C, Q4.2, U3.1
- new net VIN4: D10.C, Q5.2, U4.1
- new net VIN5: D12.C, Q6.2, U5.1
- new net VIN6: D14.C, Q7.2, U6.1
- new net VIN7: D16.C, Q8.2, U7.1
- new net V_BATT: J2.6, Q1.3
- new net V_BATT1: J7.6, Q2.3
- new net V_BATT2: J11.6, Q3.3
- new net V_BATT3: J15.6, Q4.3
- new net V_BATT4: J19.6, Q5.3
- new net V_BATT5: J23.6, Q6.3
- new net V_BATT6: J27.6, Q7.3
- new net V_BATT7: J31.6, Q8.3
- new net V_USB: D5.A, J2.4, Q1.1, R10.2
- new net V_USB1: D2.A, J7.4, Q2.1, R2.2
- new net V_USB2: D6.A, J11.4, Q3.1, R4.2
- new net V_USB3: D8.A, J15.4, Q4.1, R6.2
- new net V_USB4: D10.A, J19.4, Q5.1, R8.2
- new net V_USB5: D12.A, J23.4, Q6.1, R12.2
- new net V_USB6: D14.A, J27.4, Q7.1, R14.2
- new net V_USB7: D16.A, J31.4, Q8.1, R16.2
- net 3.3V: now also JP2.2, U$3.14; no longer J4.7, U$22.14, U$22.15
- net 3.3V1: now also JP4.2, U$34.14; no longer J6.7, U$23.14, U$23.15
- net 3.3V2: now also JP6.2, U$53.14; no longer J9.7, U$43.14, U$43.15
- net 3.3V3: now also JP8.2, U$72.14; no longer J12.7, U$58.14, U$58.15
- net 3.3V4: now also JP10.2, U$91.14; no longer J15.7, U$73.14, U$73.15
- net 3.3V5: now also JP12.2, U$110.14; no longer J18.7, U$88.14, U$88.15
- net 3.3V6: now also JP14.2, U$129.14; no longer J21.7, U$103.14, U$103.15
- net 3.3V7: now also JP16.2, U$148.14; no longer J24.7, U$118.14, U$118.15
- net BOOT: now also U$3.3; no longer U$22.3
- net BOOT1: now also J8.4, U$34.3; no longer J2.4, U$23.3
- net BOOT2: now also J12.4, U$53.3; no longer J7.4, U$43.3
- net BOOT3: now also J16.4, U$72.3; no longer J10.4, U$58.3
- net BOOT4: now also J20.4, U$91.3; no longer J13.4, U$73.3
- net BOOT5: now also J24.4, U$110.3; no longer J16.4, U$88.3
- net BOOT6: now also J28.4, U$129.3; no longer J19.4, U$103.3
- net BOOT7: now also J32.4, U$148.3; no longer J22.4, U$118.3
- net CIPO: now also U$3.10; no longer U$22.10
- net CIPO1: now also U$34.10; no longer U$23.10
- net CIPO2: now also J9.4, U$53.10; no longer J8.4, U$43.10
- net CIPO3: now also J13.4, U$72.10; no longer J11.4, U$58.10
- net CIPO4: now also J17.4, U$91.10; no longer J14.4, U$73.10
- net CIPO5: now also J21.4, U$110.10; no longer J17.4, U$88.10
- net CIPO6: now also J25.4, U$129.10; no longer J20.4, U$103.10
- net CIPO7: now also J29.4, U$148.10; no longer J23.4, U$118.10
- net COPI: now also U$3.9; no longer U$22.9
- net COPI1: now also U$34.9; no longer U$23.9
- net COPI2: now also J9.5, U$53.9; no longer J8.5, U$43.9
- net COPI3: now also J13.5, U$72.9; no longer J11.5, U$58.9
- net COPI4: now also J17.5, U$91.9; no longer J14.5, U$73.9
- net COPI5: now also J21.5, U$110.9; no longer J17.5, U$88.9
- net COPI6: now also J25.5, U$129.9; no longer J20.5, U$103.9
- net COPI7: now also J29.5, U$148.9; no longer J23.5, U$118.9
- net CS: now also U$3.7; no longer U$22.7
- net CS1: now also U$34.7; no longer U$23.7
- net CS2: now also J9.7, U$53.7; no longer J8.7, U$43.7
- net CS3: now also J13.7, U$72.7; no longer J11.7, U$58.7
- net CS4: now also J17.7, U$91.7; no longer J14.7, U$73.7
- net CS5: now also J21.7, U$110.7; no longer J17.7, U$88.7
- net CS6: now also J25.7, U$129.7; no longer J20.7, U$103.7
- net CS7: now also J29.7, U$148.7; no longer J23.7, U$118.7
- net G1: now also J8.3, U$34.1; no longer J2.3, U$23.1
- net G2: now also J12.3, U$53.1; no longer J7.3, U$43.1
- net G3: now also J16.3, U$72.1; no longer J10.3, U$58.1
- net G4: now also J20.3, U$91.1; no longer J13.3, U$73.1
- net G5: now also J24.3, U$110.1; no longer J16.3, U$88.1
- net G6: now also J28.3, U$129.1; no longer J19.3, U$103.1
- net G7: now also J32.3, U$148.1; no longer J22.3, U$118.1
- net G8: now also U$3.1; no longer U$22.1
- net GND: now also C47.2, R10.1, U$3.12, U$3.13, U$3.22, U$3.24, U8.2; no longer C2.2, C45.2, U$22.12, U$22.16, U$22.22, U$22.24, U1.4
- net GND1: now also R2.1, U$34.12, U$34.13, U$34.22, U$34.24, U1.2; no longer C3.2, U$23.12, U$23.16, U$23.22, U$23.24, U2.4
- net GND2: now also C2.2, D3.C, J10.5, R4.1, U$53.12, U$53.13, U$53.22, U$53.24, U2.2; no longer C4.2, C5.2, D2.C, J9.5, U$43.12, U$43.16, U$43.22, U$43.24, U3.4
- net GND3: now also C3.2, D7.C, J14.5, R6.1, U$72.12, U$72.13, U$72.22, U$72.24, U3.2; no longer C6.2, C7.2, D3.C, J12.5, U$58.12, U$58.16, U$58.22, U$58.24, U4.4
- net GND4: now also C4.2, D9.C, J18.5, R8.1, U$91.12, U$91.13, U$91.22, U$91.24, U4.2; no longer C8.2, C9.2, D5.C, J15.5, U$73.12, U$73.16, U$73.22, U$73.24, U5.4
- net GND5: now also C5.2, D11.C, J22.5, R12.1, U$110.12, U$110.13, U$110.22, U$110.24, U5.2; no longer C10.2, C11.2, D6.C, J18.5, U$88.12, U$88.16, U$88.22, U$88.24, U6.4
- net GND6: now also C6.2, D13.C, J26.5, R14.1, U$129.12, U$129.13, U$129.22, U$129.24, U6.2; no longer C12.2, C13.2, D7.C, J21.5, U$103.12, U$103.16, U$103.22, U$103.24, U7.4
- net GND7: now also C7.2, D15.C, J30.5, R16.1, U$148.12, U$148.13, U$148.22, U$148.24, U7.2; no longer C14.2, C15.2, D8.C, J24.5, U$118.12, U$118.16, U$118.22, U$118.24, U8.4
- net INT1: now also U$3.4; no longer U$22.4
- net INT10: now also J20.5, U$91.4; no longer J13.5, U$73.4
- net INT11: now also J24.6, U$110.5; no longer J16.6, U$88.5
- net INT12: now also J24.5, U$110.4; no longer J16.5, U$88.4
- net INT13: now also J28.6, U$129.5; no longer J19.6, U$103.5
- net INT14: now also J28.5, U$129.4; no longer J19.5, U$103.4
- net INT15: now also J32.6, U$148.5; no longer J22.6, U$118.5
- net INT16: now also J32.5, U$148.4; no longer J22.5, U$118.4
- net INT2: now also U$3.5; no longer U$22.5
- net INT3: now also J8.6, U$34.5; no longer J2.6, U$23.5
- net INT4: now also J8.5, U$34.4; no longer J2.5, U$23.4
- net INT5: now also J12.6, U$53.5; no longer J7.6, U$43.5
- net INT6: now also J12.5, U$53.4; no longer J7.5, U$43.4
- net INT7: now also J16.6, U$72.5; no longer J10.6, U$58.5
- net INT8: now also J16.5, U$72.4; no longer J10.5, U$58.4
- net INT9: now also J20.6, U$91.5; no longer J13.6, U$73.5
- net N$1: now also D1.A, R1.1; no longer E1.SIG, U$22.23
- net N$2: now also D3.A, R3.1; no longer R2.1, U1.7
- net N$3: now also D7.A, R5.1; no longer R11.1, U1.3
- net N$4: now also D9.A, R7.1; no longer R1.1, U2.7
- net N$5: now also D11.A, R11.1; no longer R3.1, U2.3
- net N$6: now also D13.A, R13.1; no longer D1.A, R4.1
- net N$7: now also D15.A, R15.1; no longer E2.SIG, U$23.23
- net PWR_EN: now also J2.2, U$3.15; no longer J1.8, U$22.13
- net PWR_EN1: now also J7.2, U$34.15; no longer J2.8, U$23.13
- net PWR_EN2: now also J11.2, U$53.15; no longer J7.8, U$43.13
- net PWR_EN3: now also J15.2, U$72.15; no longer J10.8, U$58.13
- net PWR_EN4: now also J19.2, U$91.15; no longer J13.8, U$73.13
- net PWR_EN5: now also J23.2, U$110.15; no longer J16.8, U$88.13
- net PWR_EN6: now also J27.2, U$129.15; no longer J19.8, U$103.13
- net PWR_EN7: now also J31.2, U$148.15; no longer J22.8, U$118.13
- net RESETB: now also J2.1, U$3.6; no longer J1.7, U$22.6
- net RESETB1: now also J7.1, U$34.6; no longer J2.7, U$23.6
- net RESETB2: now also J11.1, U$53.6; no longer J7.7, U$43.6
- net RESETB3: now also J15.1, U$72.6; no longer J10.7, U$58.6
- net RESETB4: now also J19.1, U$91.6; no longer J13.7, U$73.6
- net RESETB5: now also J23.1, U$110.6; no longer J16.7, U$88.6
- net RESETB6: now also J27.1, U$129.6; no longer J19.7, U$103.6
- net RESETB7: now also J31.1, U$148.6; no longer J22.7, U$118.6
- net SCLK: now also U$3.8; no longer U$22.8
- net SCLK1: now also U$34.8; no longer U$23.8
- net SCLK2: now also J9.6, U$53.8; no longer J8.6, U$43.8
- net SCLK3: now also J13.6, U$72.8; no longer J11.6, U$58.8
- net SCLK4: now also J17.6, U$91.8; no longer J14.6, U$73.8
- net SCLK5: now also J21.6, U$110.8; no longer J17.6, U$88.8
- net SCLK6: now also J25.6, U$129.8; no longer J20.6, U$103.8
- net SCLK7: now also J29.6, U$148.8; no longer J23.6, U$118.8
Routing:
- net VDD7: track 40.0 -> 0.00 mm, vias 3 -> 0
- net VDD3: track 40.0 -> 0.00 mm, vias 3 -> 0
- net VDD5: track 40.0 -> 0.00 mm, vias 3 -> 0
- net VDD4: track 40.0 -> 0.00 mm, vias 3 -> 0
- net VDD1: track 40.0 -> 0.00 mm, vias 3 -> 0
- net VDD: track 40.0 -> 0.00 mm, vias 3 -> 0
- net VDD6: track 40.0 -> 0.00 mm, vias 3 -> 0
- net VDD2: track 40.0 -> 0.00 mm, vias 3 -> 0
- net FLSH_SI7: track 29.6 -> 0.00 mm
- net FLSH_SI3: track 29.6 -> 0.00 mm
- net FLSH_SI5: track 29.6 -> 0.00 mm
- net FLSH_SI1: track 29.6 -> 0.00 mm
- net FLSH_SI4: track 29.6 -> 0.00 mm
- net FLSH_SI6: track 29.6 -> 0.00 mm
- net FLSH_SI: track 29.6 -> 0.00 mm
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